File: Bast-M7/Bast-M7.sch (KiCad schematic (older format))
At the start: 39 parts

Commit message: USB pins
Connections:
- wire segments 136 -> 140
Changed lines of the file:
@@
 Text Label 3880 1830 0    50   ~ 0
 SWCLK
+Wire Wire Line
+	3670 2130 3880 2130
+Wire Wire Line
+	3670 2030 3870 2030
+Wire Wire Line
+	3670 1430 3890 1430
+Wire Wire Line
+	3670 1530 3890 1530
 $EndSCHEMATC

Commit message: Update SPI Flash, GPIOs, Analog pins, SPI, I2C and Serial
Parts:
- added J1: Conn_Battery, Connector_JST:JST_PH_B2B-PH-SM4-TB_1x02-1MP_P2.00mm_Vertical, symbol Connector_Generic:Conn_02x01
- added J3: Conn_Left, Connector_PinSocket_2.54mm:PinSocket_1x16_P2.54mm_Vertical, symbol Connector_Generic:Conn_01x16
- added J4: Conn_Right, Connector_PinSocket_2.54mm:PinSocket_1x12_P2.54mm_Vertical, symbol Connector_Generic:Conn_01x12
- added P1: USB_C_Plug_USB2.0, symbol Connector:USB_C_Plug_USB2.0
- added R1, R3: 10K, symbol Device:R_Small
- added R4: 33K, symbol Device:R_Small
- added R5, R6: 5.1K, symbol Device:R_Small
- added SW1, SW2: RESET, symbol Switch:SW_Push
- added U1: W25Q128JVS, Package_SO:SOIC-8_5.23x5.23mm_P1.27mm, symbol Memory_Flash:W25Q128JVS
- gave numbers to parts that had none: 39
Connections:
- net labels added: +3.3V, +BATT, A0, A1, A2, A3, A4, A5, Aref, CS, D+, D-, EN, FlexSPI_CLK_A, FlexSPI_D0_A, FlexSPI_D1_A, FlexSPI_D2_A, FlexSPI_D3_A, FlexSPI_SS0, GPIO05, GPIO06, GPIO09, GPIO10, GPIO11, GPIO12, GPIO13, GPIO5, GPIO6, GPIO9, MISC, MISO, MOSI, ONOFF, POR_BUTTONENABLE, RX, SCK, SCL, SDA, TX, VBUS, ~RST~
- wire segments 140 -> 201
- no-connect marks 0 -> 13
Other:
- note added: "BATTERY CHARGER"
- note added: "FEATHER CONNECTOR"
- note added: "QSPI FLASH"
- note added: "REGULATOR"
- note added: "RESET AND MISSELANIUS"
- moved on the sheet: C1, C10, C11, C12, C13, C14, C15, C16, C17, C18, C19, C2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

Commit message: Charger battery, fix Serial, and Boot pins
Parts:
- removed U3: AP2112K-3.3, Package_TO_SOT_SMD:SOT-23-5, symbol Regulator_Linear:AP2112K-3.3
- added C34, C35: 10uF, symbol Device:C_Small
- added C36: 4.7uH, symbol Device:C_Small
- added C37: 22uF, symbol Device:C_Small
- added C38: C_Small, symbol Device:C_Small
- added D1, D3: LED, symbol Device:LED
- added D2: MBR340, Diode_THT:D_DO-201AD_P15.24mm_Horizontal, symbol Diode:MBR340
- added L2: 100nF, symbol Device:L_Small
- added Q1: TP0610L, Package_TO_SOT_THT:TO-92L_Inline, symbol Transistor_FET:TP0610L
- added R10: 10K, symbol Device:R_Small
- added R11: 330, symbol Device:R_Small
- added R7: 1K, symbol Device:R_Small
- added R8: 1k, symbol Device:R_Small
- added R9: R_Small, symbol Device:R_Small
- added U3: MCP73831-3-OT, Package_TO_SOT_SMD:SOT-23-5, symbol Battery_Management:MCP73831-3-OT
- added U4: AP63203WU-7, Package_TO_SOT_SMD:TSOT-23-6, symbol Regulator_Switching:AP63203WU-7
- SW1: value RESET -> ENABLE
Connections:
- net labels added: BOOT0, BOOT1, BOOT2, BOOT3, LED, RST
- net labels removed: CS, GPIO5, GPIO6, GPIO9, POR_BUTTONENABLE, ~RST~
- wire segments 201 -> 239
- no-connect marks 13 -> 12
Other:
- moved on the sheet: C13, C16, J1, J3, J4, P1, R1, R3, R4, R5, R6, U1

Commit message: boot, swconn and another connections added
Parts:
- added C39, C40, C41: 1uF, symbol Device:C
- added C42: 220nF, symbol Device:C
- added J2: SWD, symbol Connector:Screw_Terminal_01x04
- added JP1: Jumper_3_Bridged12, symbol Jumper:Jumper_3_Bridged12
- added R12, R13, R14, R15: 1K, symbol Device:R_Small
- added R16, R17, R18, R19, R20: 10K, symbol Device:R_Small
- added SW3: SW_DIP_x04, symbol Switch:SW_DIP_x04
- added SW4: RESET, symbol Switch:SW_Push
- SW2: value RESET -> ONOFF
- U2: symbol MCU_NXP_RT:MIMXRT1011DAE5A -> Bast-M7-rescue:MIMXRT1011DAE5A-MCU_NXP_RT
- U4: symbol Regulator_Switching:AP63203WU-7 -> Bast-M7-rescue:AP63203WU-7-Regulator_Switching
Connections:
- net labels added: PMIC, POR_B, VDDA
- net labels removed: MISC, RST
- wire segments 239 -> 297
- no-connect marks 12 -> 13
Other:
- moved on the sheet: D3, R11, SW1, SW2

Commit message: boot fixed
Parts:
- added R? (x2): 47K, symbol Device:R_Small
- JP1: value Jumper_3_Bridged12 -> ArefJmp
- R16, R17, R18, R19: value 10K -> 47K
Connections:
- net +3V3: now also C11.1, C8.1, U2.31 (VDD_USB_CAP)
- net BOOT0: now also U2.74 (GPIO_SD_02), R?.1; no longer U2.76 (GPIO_SD_00)
- net BOOT2: now also U2.76 (GPIO_SD_00); no longer R17.1, SW3.6, U2.74 (GPIO_SD_02)
- net BOOT3: now also R?.1; no longer R16.1, SW3.5
- net GND: now also R?.2, R?.2
- net BOOT_M0: now reaches U2.72 (GPIO_SD_04)
- net BOOT_M0: now also R16.1, SW3.5
- net BOOT_M1: now reaches U2.73 (GPIO_SD_03)
- net BOOT_M1: now also R17.1, SW3.6
- no-connect marks 13 -> 11
Other:
- moved on the sheet: C41, R16, R17, R18, R19, SW1

Commit message: nvcc and some capacitors fixed
Parts:
- added C? (x2): 100nF, symbol Device:C_Small
- added D?: RB521S30, symbol Device:D_Schottky
- C25, C27: value 0.22uF -> 4.7uF
- C31, C33: value 0.22uF -> 100nF
Connections:
- net +3V3: now also C5.1, C7.1, U2.39 (VDD_HIGH_IN), C?.1, C?.1, D?.2 (A); no longer R2.2, U2.31 (VDD_USB_CAP)
- net GND: now also C20.2, C25.2, C27.2, C29.2, C31.2, C33.2, C5.2, C7.2, C?.2, C?.2; no longer C20.1, C5.1, C7.1
- net VDD_SNVS_IN: now reaches U2.25 (VDD_SNVS_IN)
- net VDD_SNVS_IN: now also C20.1, D?.1 (K); no longer C20.2
- net at U2.26 (VDD_SNVS_CAP): no longer C1.1
- net at C13.1, C16.1: no longer U2.35 (VDD_HIGH_CAP)
- net at C15.1, C19.1: no longer U2.40 (NVCC_PLL)
- new net: C23.1, R2.1
- now unconnected: L1.2, U2.15 (DCDC_PSWITCH), U2.19 (DCDC_LP)
Other:
- moved on the sheet: C10, C14, C17, C18, C2, C20, C21, C22, C23, C25, C27, C29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

Commit message: fixed some pin configurations and capacitors
Parts:
- removed C18: 22uF, symbol Device:C_Small
- added C?: 22uF, symbol Device:C_Small
- C38_10V: renamed from C38; value C_Small -> 1uF
Connections:
- net +3V3: now also R2.2, U2.31 (VDD_USB_CAP)
- net DCDC_OUT: now also C?.1
- net GND: now also C24.2, C26.2, C28.2, C30.2, C32.2, C?.2
- net DCDC_PSWITCH: now reaches U2.15 (DCDC_PSWITCH)
- net DCDC_PSWITCH: now also C23.1, R2.1
- net DCDC_LP: now reaches U2.19 (DCDC_LP)
- net DCDC_LP: now also L1.2
- net VDD_SNVS_CAP: now reaches U2.26 (VDD_SNVS_CAP)
- net VDD_SNVS_CAP: now also C1.1
- net VDD_HIGH_CAP: now reaches U2.35 (VDD_HIGH_CAP)
- net VDD_HIGH_CAP: now also C13.1, C16.1
- net NVCC_PLL: now reaches U2.40 (NVCC_PLL)
- net NVCC_PLL: now also C15.1, C19.1
Other:
- moved on the sheet: C1, C11, C12, C13, C14, C15, C16, C17, C19, C2, C21, C23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

Commit message: reset and other changes
Parts:
- removed C40: 1uF, symbol Device:C
- removed SW4: RESET, symbol Switch:SW_Push
- added J?: TEST RESET, symbol Connector_Generic:Conn_02x04_Counter_Clockwise
- SW1: value ENABLE -> RESET
Connections:
- net +3V3: now also J?.4 (Pin_4)
- net GND: now also P1.S1 (SHIELD), J?.5 (Pin_5)
- net EN renamed Both
- net Both: now also J?.6 (Pin_6), J?.7 (Pin_7), J?.8 (Pin_8); no longer C41.1, SW1.2
- new net rst: C41.1, J?.1 (Pin_1), J?.2 (Pin_2), J?.3 (Pin_3), SW1.2
- no-connect marks 11 -> 10
Other:
- note added: "BOOT\n"
- note added: "CAPACITORS\n"
- note added: "MICROCONTROLLER\n"
- note added: "OSCILLATORS"
- note added: "RESET AND MISCELLANEOUS"
- note added: "SWD CONNECTOR"
- note added: "USB C"
- note added: "VREF JUMPER\n"
- note removed: "RESET AND MISSELANIUS"
- moved on the sheet: C1, C10, C11, C12, C13, C14, C15, C16, C17, C19, C2, C20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
